File: PCB/Thinpact.kicad_pcb (KiCad board)
At the start: 2 copper layers, 228.6 x 116.7 mm, 129 parts, among them SW1 SW_PUSH, SW10 SW_PUSH, SW11 SW_PUSH, SW12 SW_PUSH, SW13 SW_PUSH, SW14 SW_PUSH, SW15 SW_PUSH, SW16 SW_PUSH, SW17 SW_PUSH, SW18 SW_PUSH, SW19 SW_PUSH, SW2 SW_PUSH, SW20 SW_PUSH, SW21 SW_PUSH, SW22 SW_PUSH, SW23 SW_PUSH, SW24 SW_PUSH, SW25 SW_PUSH, SW26 SW_PUSH, SW27 SW_PUSH, SW28 SW_PUSH, SW29 SW_PUSH, SW3 SW_PUSH, SW30 SW_PUSH, SW31 SW_PUSH, SW32 SW_PUSH, SW33 SW_PUSH, SW34 SW_PUSH, SW35 SW_PUSH, SW36 SW_PUSH, SW37 SW_PUSH, SW38 SW_PUSH, SW39 SW_PUSH, SW4 SW_PUSH, SW40 SW_PUSH, SW41 SW_PUSH, SW42 SW_PUSH, SW43 SW_PUSH, SW44 SW_PUSH, SW45 SW_PUSH, SW46 SW_PUSH, SW47 SW_PUSH, SW48 SW_PUSH, SW49 SW_PUSH, SW5 SW_PUSH, SW50 SW_PUSH, SW51 SW_PUSH, SW52 SW_PUSH, SW53 SW_PUSH, SW54 SW_PUSH, SW55 SW_PUSH, SW56 SW_PUSH, SW57 SW_PUSH, SW58 SW_PUSH, SW59 SW_PUSH, SW6 SW_PUSH, SW60 SW_SPDT, SW61 SW_SPDT, SW7 SW_PUSH, SW8 SW_PUSH, SW9 SW_PUSH, U1 Micon_BLEMicroPro, U2 Micon_BLEMicroPro

Commit message: Update sch and kicad_pcb
Parts:
- SW1, SW2, SW3, SW4: footprint footprints:Choc_Hotswap_1u -> footprints:Choc_Hotswap_1u_Small
Connections:
- U1 pad 21: VCC -> unconnected-(U1-VCC-Pad21)
- U2 pad 21: VCC -> unconnected-(U2-VCC-Pad21)
Changed lines of the file:
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@@
 	(net 5 "col5")
 	(net 6 "row3")
-	(net 7 "VCC")
+	(net 7 "unconnected-(U2-VCC-Pad21)")
 	(net 8 "row9")
 	(net 9 "col0")
@@
 	(net 89 "unconnected-(SW60-C-Pad3)")
 	(net 90 "Net-(D61-A)")
+	(net 91 "unconnected-(U1-VCC-Pad21)")
 	(footprint "footprints:Choc_Hotswap_1u"
 		(layer "F.Cu")
@@
 			(layers "*.Cu" "*.Mask" "F.SilkS")
 			(remove_unused_layers no)
-			(net 7 "VCC")
+			(net 7 "unconnected-(U2-VCC-Pad21)")
 			(pinfunction "VCC")
-			(pintype "power_in")
+			(pintype "power_in+no_connect")
 		)
 		(pad "22" thru_hole circle
@@
 		(embedded_fonts no)
 	)
-	(footprint "footprints:Choc_Hotswap_1u"
+	(footprint "footprints:Choc_Hotswap_1u_Small"
 		(layer "F.Cu")
 		(at 38.1 90.4875)
-		(descr "Supported: Choc v1/v2, hotswap, 1u")
+		(descr "Supported: Choc v1/v2, hotswap, 1u. This is for edge-located key switches.")
 		(property "Reference" "SW2"
 			(at -5.08 -6.35 180)
@@
 		)
 		(pad "1" smd rect
-			(at -8.575 3.7 180)
-			(size 2.6 2.6)
+			(at -8.175 3.7 180)
+			(size 1.8 3)
 			(layers "B.Cu" "B.Mask" "B.Paste")
 			(net 9 "col0")
@@
 		)
 	)
-	(footprint "footprints:Choc_Hotswap_1u"
+	(footprint "footprints:Choc_Hotswap_1u_Small"
 		(layer "F.Cu")
 		(at 38.1 109.5375)
-		(descr "Supported: Choc v1/v2, hotswap, 1u")
+		(descr "Supported: Choc v1/v2, hotswap, 1u. This is for edge-located key switches.")
 		(property "Reference" "SW3"
 			(at -5.08 -6.35 180)
@@
 		)
 		(pad "1" smd rect
-			(at -8.575 3.7 180)
-			(size 2.6 2.6)
+			(at -8.175 3.7 180)
+			(size 1.8 3)
 			(layers "B.Cu" "B.Mask" "B.Paste")
 			(net 9 "col0")
@@
 		(embedded_fonts no)
 	)
-	(footprint "footprints:Choc_Hotswap_1u"
+	(footprint "footprints:Choc_Hotswap_1u_Small"
 		(layer "F.Cu")
 		(at 38.1 71.4375)
-		(descr "Supported: Choc v1/v2, hotswap, 1u")
+		(descr "Supported: Choc v1/v2, hotswap, 1u. This is for edge-located key switches.")
 		(property "Reference" "SW1"
 			(at -5.08 -6.35 180)
@@
 		)
 		(pad "1" smd rect
-			(at -8.575 3.7 180)
-			(size 2.6 2.6)
+			(at -8.175 3.7 180)
+			(size 1.8 3)
 			(layers "B.Cu" "B.Mask" "B.Paste")
 			(net 9 "col0")
@@
 			(layers "*.Cu" "*.Mask" "F.SilkS")
 			(remove_unused_layers no)
-			(net 7 "VCC")
+			(net 91 "unconnected-(U1-VCC-Pad21)")
 			(pinfunction "VCC")
-			(pintype "power_in")
+			(pintype "power_in+no_connect")
 		)
 		(pad "22" thru_hole circle
@@
 		)
 	)
-	(footprint "footprints:Choc_Hotswap_1u"
+	(footprint "footprints:Choc_Hotswap_1u_Small"
 		(layer "F.Cu")
 		(at 38.1 128.5875)
-		(descr "Supported: Choc v1/v2, hotswap, 1u")
+		(descr "Supported: Choc v1/v2, hotswap, 1u. This is for edge-located key switches.")
 		(property "Reference" "SW4"
 			(at -5.08 -6.35 180)
@@
 		)
 		(pad "1" smd rect
-			(at -8.575 3.7 180)
-			(size 2.6 2.6)
+			(at -8.175 3.7 180)
+			(size 1.8 3)
 			(layers "B.Cu" "B.Mask" "B.Paste")
 			(net 9 "col0")

Commit message: Circuit patterns for v0.0.1
Parts:
- added H1: H, kbd_Hole:m2_Screw_Hole, F.Cu at (33.3, 50.0)
- added H10: H, kbd_Hole:m2_Spacer_Hole_hex, F.Cu at (104.8, 119.1)
- added H11: H, kbd_Hole:m2_Spacer_Hole_hex, F.Cu at (142.9, 119.1)
- added H12: H, kbd_Hole:m2_Spacer_Hole_hex, F.Cu at (181.0, 119.1)
- added H13: H, kbd_Hole:m2_Spacer_Hole_hex, F.Cu at (238.1, 119.1)
- added H14: H, kbd_Hole:m2_Spacer_Hole_hex, F.Cu at (96.4, 141.1)
- added H15: H, kbd_Hole:m2_Spacer_Hole_hex, F.Cu at (189.3, 141.1)
- added H16: H, kbd_Hole:m2_Spacer_Hole_hex, F.Cu at (142.9, 147.6)
- added H2: H, kbd_Hole:m2_Screw_Hole, F.Cu at (142.9, 50.0)
- added H3: H, kbd_Hole:m2_Screw_Hole, F.Cu at (252.4, 50.0)
- added H4: H, kbd_Hole:m2_Spacer_Hole_hex, F.Cu at (47.6, 81.0)
- added H5: H, kbd_Hole:m2_Spacer_Hole_hex, F.Cu at (104.8, 81.0)
- added H6: H, kbd_Hole:m2_Spacer_Hole_hex, F.Cu at (142.9, 81.0)
- added H7: H, kbd_Hole:m2_Spacer_Hole_hex, F.Cu at (181.0, 81.0)
- added H8: H, kbd_Hole:m2_Spacer_Hole_hex, F.Cu at (238.1, 81.0)
- added H9: H, kbd_Hole:m2_Spacer_Hole_hex, F.Cu at (47.6, 119.1)
- SW9: footprint footprints:Choc_Hotswap_1u -> footprints:Choc_Hotswap_1u_Small
- moved JP1 5.82 mm to (90.8, 49.0), turned to -90 degrees
- moved D59 4.41 mm to (149.6, 48.8)
- moved BT1 3.98 mm to (163.4, 49.3)
- moved BT2 3.98 mm to (194.4, 49.3)
- moved D60 3.98 mm to (180.4, 48.8)
- moved D42 2.04 mm to (197.5, 113.5)
- moved D15 1.94 mm to (102.2, 75.5)
- moved D52 1.94 mm to (235.6, 113.6)
- moved D53 1.89 mm to (235.6, 132.7)
- moved D37 1.84 mm to (178.4, 113.7)
- moved D1 1.83 mm to (45.1, 75.6)
- moved D17 1.74 mm to (102.2, 113.8)
- moved D25 1.74 mm to (140.3, 75.7)
- moved D27 1.74 mm to (140.3, 113.8)
- moved D50 1.74 mm to (235.6, 75.7)
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Routing:
- net col0: track 0.00 -> 433.1 mm, vias 0 -> 3
- net col2: track 0.00 -> 432.4 mm, vias 0 -> 3
- net col1: track 0.00 -> 411.4 mm, vias 0 -> 2
- net row5: track 0.00 -> 403.0 mm, vias 0 -> 6
- net col3: track 0.00 -> 400.9 mm, vias 0 -> 7
- net col4: track 0.00 -> 400.1 mm, vias 0 -> 3
- net row6: track 0.00 -> 393.4 mm, vias 0 -> 1
- net row8: track 0.00 -> 392.3 mm, vias 0 -> 7
- net row9: track 0.00 -> 391.7 mm, vias 0 -> 2
- net col5: track 0.00 -> 380.1 mm, vias 0 -> 3
- net row7: track 0.00 -> 376.1 mm, vias 0 -> 6
- net row4: track 0.00 -> 364.7 mm, vias 0 -> 8
- net row3: track 0.00 -> 323.4 mm, vias 0 -> 6
- net row1: track 0.00 -> 300.3 mm, vias 0 -> 7
- net row0: track 0.00 -> 267.3 mm, vias 0 -> 8
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- added copper zone on B.Cu, net GND
- added copper zone on F.Cu, net GND
Other:
- board text added: "Craft Keyboard main board 2025/5/11 Ver. 0.0.1"
