File: PCB/Thinpact.kicad_sch (KiCad schematic)
At the start: 129 parts, among them SW1 SW_PUSH, SW10 SW_PUSH, SW11 SW_PUSH, SW12 SW_PUSH, SW13 SW_PUSH, SW14 SW_PUSH, SW15 SW_PUSH, SW16 SW_PUSH, SW17 SW_PUSH, SW18 SW_PUSH, SW19 SW_PUSH, SW2 SW_PUSH, SW20 SW_PUSH, SW21 SW_PUSH, SW22 SW_PUSH, SW23 SW_PUSH, SW24 SW_PUSH, SW25 SW_PUSH, SW26 SW_PUSH, SW27 SW_PUSH, SW28 SW_PUSH, SW29 SW_PUSH, SW3 SW_PUSH, SW30 SW_PUSH, SW31 SW_PUSH, SW32 SW_PUSH, SW33 SW_PUSH, SW34 SW_PUSH, SW35 SW_PUSH, SW36 SW_PUSH, SW37 SW_PUSH, SW38 SW_PUSH, SW39 SW_PUSH, SW4 SW_PUSH, SW40 SW_PUSH, SW41 SW_PUSH, SW42 SW_PUSH, SW43 SW_PUSH, SW44 SW_PUSH, SW45 SW_PUSH, SW46 SW_PUSH, SW47 SW_PUSH, SW48 SW_PUSH, SW49 SW_PUSH, SW5 SW_PUSH, SW50 SW_PUSH, SW51 SW_PUSH, SW52 SW_PUSH, SW53 SW_PUSH, SW54 SW_PUSH, SW55 SW_PUSH, SW56 SW_PUSH, SW57 SW_PUSH, SW58 SW_PUSH, SW59 SW_PUSH, SW6 SW_PUSH, SW60 SW_SPDT, SW61 SW_SPDT, SW7 SW_PUSH, SW8 SW_PUSH, SW9 SW_PUSH, U1 Micon_BLEMicroPro, U2 Micon_BLEMicroPro

Commit message: Update sch and kicad_pcb(not routed)
Parts:
- BT1, BT2: footprint kbd_Parts:Battery_ali_CR1632 -> footprints:HU1632
- C1: footprint kbd_Parts:Capacitor_1206 -> Capacitor_SMD:C_1206_3216Metric_Pad1.33x1.80mm_HandSolder
- D1, D10, D11, D12, D13, D14, D15, D16, D17, D18, D19, D2, D20, D21, D22, D23, D24, D25, D26, D27, D28, D29, D3, D30, D31, D32, D33, D34, D35, D36, D37, D38, D39, D4, D40, D41, D42, D43, D44, D45, D46, D47, D48, D49, D5, D50, D51, D52, D53, D54, D55, D56, D57, D58, D59, D6, D60, D7, D8, D9: footprint Diode_SMD:D_0603_1608Metric -> kbd_Parts:Diode_SMD
- R1: footprint Resistor_THT:R_Axial_DIN0207_L6.3mm_D2.5mm_P7.62mm_Horizontal -> Resistor_THT:R_Axial_DIN0204_L3.6mm_D1.6mm_P1.90mm_Vertical
- SW1, SW10, SW11, SW12, SW13, SW14, SW15, SW16, SW17, SW18, SW19, SW2, SW20, SW21, SW22, SW23, SW25, SW26, SW27, SW28, SW3, SW30, SW31, SW32, SW33, SW35, SW36, SW37, SW38, SW4, SW40, SW41, SW42, SW43, SW44, SW45, SW46, SW47, SW48, SW49, SW5, SW50, SW51, SW52, SW53, SW54, SW55, SW56, SW57, SW58, SW6, SW7, SW8, SW9: footprint kbd_SW:Choc_Hotswap_1u -> footprints:Choc_Hotswap_1u
- SW24, SW29, SW34, SW39: footprint kbd_SW:Choc_Hotswap_1.25u -> footprints:Choc_Hotswap_1.25u
- SW60: footprint Button_Switch_THT:SW_Slide-03_Wuerth-WS-SLTV_10x2.5x6.4_P2.54mm -> footprints:SK-12D11VG3
- SW61: footprint Button_Switch_THT:SW_Slide-03_Wuerth-WS-SLTV_10x2.5x6.4_P2.54mm -> footprints:SS-12D00G3
- U1, U2: footprint kbd_Parts:Micon_BMP_7sKB -> footprints:Micon_BMP

Commit message: Update sch and kicad_pcb
Parts:
- SW1, SW2, SW3, SW4: footprint footprints:Choc_Hotswap_1u -> footprints:Choc_Hotswap_1u_Small
Connections:
- net VCC: no longer names the net of U2.21 (VCC)
- net VCC: no longer U1.21 (VCC)
- no-connect marks 6 -> 8

Commit message: Circuit patterns for v0.0.1
Parts:
- SW9: footprint footprints:Choc_Hotswap_1u -> footprints:Choc_Hotswap_1u_Small
Changed lines of the file:
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@@
 			)
 		)
-		(property "Footprint" "footprints:Choc_Hotswap_1u"
+		(property "Footprint" "footprints:Choc_Hotswap_1u_Small"
 			(at 62.23 152.4 0)
 			(effects
