File: Switch_plate/Switch_plate.kicad_pcb (KiCad board)
At the start: 2 copper layers, 228.6 x 116.7 mm, 79 parts, among them P1 PinSocket_1x02_P2.54mm_Vertic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, SW1 SW_PUSH, SW10 SW_PUSH, SW11 SW_PUSH, SW12 SW_PUSH, SW13 SW_PUSH, SW14 SW_PUSH, SW15 SW_PUSH, SW16 SW_PUSH, SW17 SW_PUSH, SW18 SW_PUSH, SW19 SW_PUSH, SW2 SW_PUSH, SW20 SW_PUSH, SW21 SW_PUSH, SW22 SW_PUSH, SW23 SW_PUSH, SW24 SW_PUSH, SW25 SW_PUSH, SW26 SW_PUSH, SW27 SW_PUSH, SW28 SW_PUSH, SW29 SW_PUSH, SW3 SW_PUSH, SW30 SW_PUSH, SW31 SW_PUSH, SW32 SW_PUSH, SW33 SW_PUSH, SW34 SW_PUSH, SW35 SW_PUSH, SW36 SW_PUSH, SW37 SW_PUSH, SW38 SW_PUSH, SW39 SW_PUSH, SW4 SW_PUSH, SW40 SW_PUSH, SW41 SW_PUSH, SW42 SW_PUSH, SW43 SW_PUSH, SW44 SW_PUSH, SW45 SW_PUSH, SW46 SW_PUSH, SW47 SW_PUSH, SW48 SW_PUSH, SW49 SW_PUSH, SW5 SW_PUSH, SW50 SW_PUSH, SW51 SW_PUSH, SW52 SW_PUSH, SW53 SW_PUSH, SW54 SW_PUSH, SW55 SW_PUSH, SW56 SW_PUSH, SW57 SW_PUSH, SW58 SW_PUSH, SW6 SW_PUSH, SW7 SW_PUSH, SW8 SW_PUSH, SW9 SW_PUSH

Commit message: Circuit patterns for v0.0.1
Parts:
- removed the Ref** at (228.6, 138.7)
- removed the Ref** at (57.1, 138.7)
- moved Ref** 13.1 mm to (189.3, 141.1)
- moved Ref** 13.1 mm to (96.4, 141.1)
- moved Ref** 6.55 mm to (142.9, 147.6)
Other:
- board size 228.6 x 116.7 mm -> 228.6 x 95.2 mm
- board text added: "Craft Keyboard top board 2025/5/11 Ver. 0.0.1"
